File: 2.12 Mobile Robot/2.12 Mobile Robot.kicad_sch (KiCad schematic)
At the start: 24 parts, among them J1 Motor Control L, J2 Motor Control R, J3 GND, J4 3.3V, J5 UART, J6 5V, J7 Power IO, SW1 RST_SW, SW2 BOOT_SW, SW3 SW_PWR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

Commit message: Passed DRC
Parts:
- J1, J2: footprint (none) -> Connector_PinHeader_2.54mm:PinHeader_1x05_P2.54mm_Vertical; MPN (none) -> C492404
- J3, J4, J5, J6: MPN (none) -> C2691448
- SW1, SW2: footprint (none) -> Button_Switch_THT:SW_PUSH_6mm
- SW3: footprint Connector_JST:JST_PH_B2B-PH-SM4-TB_1x02-1MP_P2.00mm_Vertical -> 2.679:SW_500SSP1S1M6QEA; MPN C160352 -> (none); now left out of the parts list
- U1: footprint (none) -> footprints:ProS3_TH
Connections:
- net +3V3 is gone; now on net +3.3V: U1.4 (3V3)
- net DIR1R is gone; now on net DIR1_R: U1.31 (IO34)
Other:
- note added: "ENCODERS"
- note added: "Microcontroller"
- note added: "OUTPUT BUSES"
- moved on the sheet: D1, J3, J4, J5, J6, R_MOTOR1
