File: 2.12 Mobile Robot/_autosave-2.12 Mobile Robot.kicad_pcb (KiCad board)
At the start: 2 copper layers, 63 parts, among them J1 Motor Control L, J2 Motor Control R, J3 GND, J4 3.3V, J5 UART, J6 5V, J8 Power IO, Q1 DMMT5401-7-F, Q2 DMG2305UX-13, SW1 RST_SW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

Commit message: Changed some of the footprints
Parts:
- removed Cbst1: 0.1uF, Capacitor_SMD:C_0805_2012Metric
- removed Cin1: 10uF, Capacitor_SMD:C_1210_3225Metric
- removed Cout1, Cout2: 22uF, Capacitor_SMD:C_1210_3225Metric
- removed D2: Power LED, LED_SMD:LED_0603_1608Metric
- removed F2: 2A, Fuse:Fuse_1206_3216Metric
- removed J8: Power IO, TerminalBlock_Phoenix:TerminalBlock_Phoenix_MKDS-3-4-5.08_1x04_P5.08mm_Horizontal
- removed L1: 3.3uH, Inductor_SMD:L_Vishay_IHLP-4040
- removed RCs2, RSE2, R_PWR1, R_PWR2: 15k, Resistor_SMD:R_0402_1005Metric
- removed R_PWR_LED1: 1kΩ, Resistor_SMD:R_0402_1005Metric
- removed Rfbb1: 10k, Resistor_SMD:R_0402_1005Metric
- removed Rfbt1: 56.2k, Resistor_SMD:R_0402_1005Metric
- removed SW4: SW_PWR, 2.679:SW_500SSP1S1M6QEA
- removed U4: POWER_IN, 2.004:DPAK85P972X240-8N
- removed U5: TPS564208DDCT, 2.004:SOT95P280X110-6N
