File: 2.12 Mobile Robot/_autosave-2.12 Mobile Robot.kicad_sch (KiCad schematic)
At the start: 27 parts, among them J1 Motor Control R, J2 Motor Control L, J3 GND, J4 Motor Power R, J5 Battery Power, J6 Motor Power L, J7 3.3V, J8 UART, J9 5V, SW1 SW_PWR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

Commit message: Renamed stuff
Parts:
- R3: renamed from RSE1; Name (none) -> RSE1
- R4: renamed from RCs1; Name (none) -> RCs1
- renumbered R_MTR1 to R1, R_MTR2 to R2, R_MOTOR1 to R5
Changed lines of the file:
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@@
   (symbol (lib_id "Device:R_US") (at 153.035 170.18 0) (unit 1)
     (in_bom yes) (on_board yes) (dnp no)
-    (property "Reference" "R_MOTOR1" (at 160.02 172.085 0)
+    (property "Reference" "R5" (at 160.02 172.085 0)
       (effects (font (size 1.27 1.27)))
     )
@@
       (project "2.12 Mobile Robot"
         (path "/7775d959-b998-472b-ab8b-c8b5c0f34c21"
-          (reference "R_MOTOR1") (unit 1)
+          (reference "R5") (unit 1)
         )
       )
@@
   (symbol (lib_id "Device:R_Small_US") (at 27.94 170.815 0) (unit 1)
     (in_bom yes) (on_board yes) (dnp no)
-    (property "Reference" "R_MTR1" (at 30.48 168.91 0)
+    (property "Reference" "R1" (at 30.48 168.91 0)
       (effects (font (size 1.27 1.27)) (justify left))
     )
@@
       (project "2.12 Mobile Robot"
         (path "/7775d959-b998-472b-ab8b-c8b5c0f34c21"
-          (reference "R_MTR1") (unit 1)
+          (reference "R1") (unit 1)
         )
       )
@@
   (symbol (lib_id "Device:R_Small_US") (at 40.005 177.8 0) (mirror y) (unit 1)
     (in_bom yes) (on_board yes) (dnp no)
-    (property "Reference" "RSE1" (at 37.465 177.165 0)
+    (property "Reference" "R3" (at 37.465 177.165 0)
       (effects (font (size 1.27 1.27)) (justify left))
     )
@@
       (effects (font (size 1.27 1.27)) hide)
     )
-    (pin "1")
-    (pin "2")
-    (instances
-      (project "2.12 Mobile Robot"
-        (path "/7775d959-b998-472b-ab8b-c8b5c0f34c21"
-          (reference "RSE1") (unit 1)
+    (property "Name" "RSE1" (at 40.005 177.8 0)
+      (effects (font (size 1.27 1.27)) hide)
+    )
+    (pin "1")
+    (pin "2")
+    (instances
+      (project "2.12 Mobile Robot"
+        (path "/7775d959-b998-472b-ab8b-c8b5c0f34c21"
+          (reference "R3") (unit 1)
         )
       )
@@
   (symbol (lib_id "Device:R_Small_US") (at 75.565 177.8 0) (unit 1)
     (in_bom yes) (on_board yes) (dnp no) (fields_autoplaced)
-    (property "Reference" "RCs1" (at 78.105 177.165 0)
+    (property "Reference" "R4" (at 78.105 177.165 0)
       (effects (font (size 1.27 1.27)) (justify left))
     )
@@
       (effects (font (size 1.27 1.27)) hide)
     )
-    (pin "1")
-    (pin "2")
-    (instances
-      (project "2.12 Mobile Robot"
-        (path "/7775d959-b998-472b-ab8b-c8b5c0f34c21"
-          (reference "RCs1") (unit 1)
+    (property "Name" "RCs1" (at 75.565 177.8 0)
+      (effects (font (size 1.27 1.27)) hide)
+    )
+    (pin "1")
+    (pin "2")
+    (instances
+      (project "2.12 Mobile Robot"
+        (path "/7775d959-b998-472b-ab8b-c8b5c0f34c21"
+          (reference "R4") (unit 1)
         )
       )
@@
   (symbol (lib_id "power:PWR_FLAG") (at 217.805 40.005 0) (unit 1)
     (in_bom yes) (on_board yes) (dnp no)
-    (property "Reference" "#FLG05" (at 217.805 38.1 0)
+    (property "Reference" "#FLG04" (at 217.805 38.1 0)
       (effects (font (size 1.27 1.27)) hide)
     )
@@
       (project "2.12 Mobile Robot"
         (path "/7775d959-b998-472b-ab8b-c8b5c0f34c21"
-          (reference "#FLG05") (unit 1)
+          (reference "#FLG04") (unit 1)
         )
       )
@@
   (symbol (lib_id "Device:R_Small_US") (at 27.94 175.895 0) (mirror y) (unit 1)
     (in_bom yes) (on_board yes) (dnp no)
-    (property "Reference" "R_MTR2" (at 26.67 175.26 0)
+    (property "Reference" "R2" (at 26.67 175.26 0)
       (effects (font (size 1.27 1.27)) (justify left))
     )
@@
       (project "2.12 Mobile Robot"
         (path "/7775d959-b998-472b-ab8b-c8b5c0f34c21"
-          (reference "R_MTR2") (unit 1)
-        )
-      )
+          (reference "R2") (unit 1)
+        )
+      )
