File: 2.12 Mobile Robot/buck.kicad_sch (KiCad schematic)
At the start: 17 parts, among them SW4 SW_PWR, U4 POWER_IN, U5 TPS564208DDCT

Commit message: Fully routed
Parts:
- C2: renamed from Cin1; Name (none) -> Cin1
- C3: renamed from Cbst1; Name (none) -> Cbst1
- C4: renamed from Cout1; Name (none) -> Cout1
- C5: renamed from Cout2; Name (none) -> Cout2
- R29: renamed from RSE2; Name (none) -> RSE2
- R30: renamed from RCs2; Name (none) -> RCs2
- R31: renamed from Rfbt1; Name (none) -> Rfbt1
- R32: renamed from Rfbb1; Name (none) -> Rfbb1
- renumbered R_PWR_LED1 to R26, R_PWR1 to R27, R_PWR2 to R28

Commit message: Made footprints from project libraries
Parts:
- U4: footprint 2.004:DPAK85P972X240-8N -> 2.12_Mobile_Robot:DPAK85P972X240-8N
- U5: footprint 2.004:SOT95P280X110-6N -> 2.12_Mobile_Robot:SOT95P280X110-6N
Changed lines of the file:
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@@
       (effects (font (size 1.27 1.27)))
     )
-    (property "Footprint" "2.004:DPAK85P972X240-8N" (at 118.11 131.445 0)
+    (property "Footprint" "2.12_Mobile_Robot:DPAK85P972X240-8N" (at 118.11 131.445 0)
       (effects (font (size 1.27 1.27)) (justify bottom) hide)
     )
@@
       (effects (font (size 1.27 1.27)))
     )
-    (property "Footprint" "2.004:SOT95P280X110-6N" (at 193.675 89.535 0)
+    (property "Footprint" "2.12_Mobile_Robot:SOT95P280X110-6N" (at 193.675 89.535 0)
       (effects (font (size 1.27 1.27)) (justify bottom) hide)
     )

Commit message: Added silkscreen callouts and fixed resistors
Parts:
- R26, R27, R28, R29, R30, R31, R32: footprint Resistor_SMD:R_0201_0603Metric_Pad0.64x0.40mm_HandSolder -> Resistor_SMD:R_0603_1608Metric
Changed lines of the file:
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@@
       (effects (font (size 1.27 1.27)) (justify left))
     )
-    (property "Footprint" "Resistor_SMD:R_0201_0603Metric_Pad0.64x0.40mm_HandSolder" (at 210.185 111.125 0)
+    (property "Footprint" "Resistor_SMD:R_0603_1608Metric" (at 210.185 111.125 0)
       (effects (font (size 1.27 1.27)) hide)
     )
@@
       (effects (font (size 1.27 1.27)))
     )
-    (property "Footprint" "Resistor_SMD:R_0201_0603Metric_Pad0.64x0.40mm_HandSolder" (at 46.609 89.916 90)
+    (property "Footprint" "Resistor_SMD:R_0603_1608Metric" (at 46.609 89.916 90)
       (effects (font (size 1.27 1.27)) hide)
     )
@@
       (effects (font (size 1.27 1.27)) (justify left))
     )
-    (property "Footprint" "Resistor_SMD:R_0201_0603Metric_Pad0.64x0.40mm_HandSolder" (at 79.375 99.695 0)
+    (property "Footprint" "Resistor_SMD:R_0603_1608Metric" (at 79.375 99.695 0)
       (effects (font (size 1.27 1.27)) hide)
     )
@@
       (effects (font (size 1.27 1.27)) (justify left))
     )
-    (property "Footprint" "Resistor_SMD:R_0201_0603Metric_Pad0.64x0.40mm_HandSolder" (at 100.33 99.695 0)
+    (property "Footprint" "Resistor_SMD:R_0603_1608Metric" (at 100.33 99.695 0)
       (effects (font (size 1.27 1.27)) hide)
     )
@@
       (effects (font (size 1.27 1.27)) (justify left))
     )
-    (property "Footprint" "Resistor_SMD:R_0201_0603Metric_Pad0.64x0.40mm_HandSolder" (at 79.375 94.615 0)
+    (property "Footprint" "Resistor_SMD:R_0603_1608Metric" (at 79.375 94.615 0)
       (effects (font (size 1.27 1.27)) hide)
     )
@@
       (effects (font (size 1.27 1.27)) (justify left))
     )
-    (property "Footprint" "Resistor_SMD:R_0201_0603Metric_Pad0.64x0.40mm_HandSolder" (at 135.89 99.695 0)
+    (property "Footprint" "Resistor_SMD:R_0603_1608Metric" (at 135.89 99.695 0)
       (effects (font (size 1.27 1.27)) hide)
     )
@@
       (effects (font (size 1.27 1.27)) (justify left))
     )
-    (property "Footprint" "Resistor_SMD:R_0201_0603Metric_Pad0.64x0.40mm_HandSolder" (at 210.185 116.84 0)
-      (effects (font (size 1.27 1.27)) hide)
-    )
+    (property "Footprint" "Resistor_SMD:R_0603_1608Metric" (at 210.185 116.84 0)
+      (effects (font (size 1.27 1.27)) hide)
+    )

Commit message: Tentatively ready for production
Parts:
- C2: footprint Capacitor_SMD:C_1210_3225Metric -> footprint:0805_2012Metric; symbol Device:C -> jlcpcb-basic-capacitor:0805,10uF,25V,X5R; LCSC (none) -> C15850; MFG (none) -> Samsung Electro-Mechanics; MFGPN (none) -> CL21A106KAYNNNE
- D2: footprint LED_SMD:LED_0603_1608Metric -> footprint:LED0603; symbol Device:LED -> jlcpcb-diodes:0603,Green; LCSC (none) -> C72043
- R26: footprint Resistor_SMD:R_0603_1608Metric -> footprint:0603_1608Metric; symbol Device:R_US -> jlcpcb-basic-resistor:0603,1k; LCSC (none) -> C21190; MFG (none) -> UNI-ROYAL(Uniroyal Elec); MFGPN (none) -> 0603WAF1001T5E
- R27, R28: footprint Resistor_SMD:R_0603_1608Metric -> footprint:0603_1608Metric; symbol Device:R_Small_US -> jlcpcb-basic-resistor:0603,15k; LCSC (none) -> C22809; MFG (none) -> UNI-ROYAL(Uniroyal Elec); MFGPN (none) -> 0603WAF1502T5E; MPN C114661 -> (none)
- R29: footprint Resistor_SMD:R_0603_1608Metric -> footprint:0603_1608Metric; symbol Device:R_Small_US -> jlcpcb-basic-resistor:0603,15k; LCSC (none) -> C22809; MFG (none) -> UNI-ROYAL(Uniroyal Elec); MFGPN (none) -> 0603WAF1502T5E; MPN C114661 -> (none); Name RSE2 -> (none)
- R30: footprint Resistor_SMD:R_0603_1608Metric -> footprint:0603_1608Metric; symbol Device:R_Small_US -> jlcpcb-basic-resistor:0603,15k; LCSC (none) -> C22809; MFG (none) -> UNI-ROYAL(Uniroyal Elec); MFGPN (none) -> 0603WAF1502T5E; MPN C114661 -> (none); Name RCs2 -> (none)
- R31: footprint Resistor_SMD:R_0603_1608Metric -> footprint:0603_1608Metric; symbol Device:R_Small_US -> jlcpcb-basic-resistor:0603,56k; LCSC (none) -> C482887; MFG (none) -> YAGEO; MFGPN (none) -> RC0603FR-0756K2L; MPN C482887 -> (none)
- R32: footprint Resistor_SMD:R_0603_1608Metric -> footprint:0603_1608Metric; symbol Device:R_Small_US -> jlcpcb-basic-resistor:0603,10k; LCSC (none) -> C25804; MFG (none) -> UNI-ROYAL(Uniroyal Elec); MFGPN (none) -> 0603WAF1002T5E
- U5: symbol TPS564208DDCT:TPS564208DDCT -> 2.12 Symbols:TPS564208DDCT
