File: 2.12 Mobile Robot/zvd.kicad_sch (KiCad schematic)
At the start: 4 parts, among them Q1 DMMT5401-7-F, Q2 DMG2305UX-13

Commit message: Renamed stuff
Parts:
- R7: footprint Resistor_SMD:R_0402_1005Metric -> Resistor_SMD:R_0201_0603Metric_Pad0.64x0.40mm_HandSolder; MPN C144807 -> C22548
- R8: footprint Resistor_SMD:R_0402_1005Metric -> Resistor_SMD:R_0201_0603Metric_Pad0.64x0.40mm_HandSolder
Changed lines of the file:
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@@
   (symbol (lib_id "power:PWR_FLAG") (at 133.35 60.96 0) (unit 1)
     (in_bom yes) (on_board yes) (dnp no) (fields_autoplaced)
-    (property "Reference" "#FLG02" (at 133.35 59.055 0)
+    (property "Reference" "#FLG04" (at 133.35 59.055 0)
       (effects (font (size 1.27 1.27)) hide)
     )
@@
       (project "2.12 Mobile Robot"
         (path "/7775d959-b998-472b-ab8b-c8b5c0f34c21/3499523e-0988-447b-89ea-8d43c1ae7973"
-          (reference "#FLG02") (unit 1)
+          (reference "#FLG04") (unit 1)
         )
       )
@@
       (effects (font (size 1.27 1.27)) (justify left))
     )
-    (property "Footprint" "Resistor_SMD:R_0402_1005Metric" (at 114.046 89.154 90)
+    (property "Footprint" "Resistor_SMD:R_0201_0603Metric_Pad0.64x0.40mm_HandSolder" (at 114.046 89.154 90)
       (effects (font (size 1.27 1.27)) hide)
     )
@@
       (effects (font (size 1.27 1.27)) hide)
     )
-    (property "MPN" "C144807" (at 113.03 88.9 0)
+    (property "MPN" "C22548" (at 113.03 88.9 0)
       (effects (font (size 1.27 1.27)) hide)
     )
@@
       (project "2.12 Mobile Robot"
         (path "/7775d959-b998-472b-ab8b-c8b5c0f34c21/3499523e-0988-447b-89ea-8d43c1ae7973"
-          (reference "R4") (unit 1)
+          (reference "R20") (unit 1)
         )
       )
@@
       (project "2.12 Mobile Robot"
         (path "/7775d959-b998-472b-ab8b-c8b5c0f34c21/3499523e-0988-447b-89ea-8d43c1ae7973"
-          (reference "#PWR044") (unit 1)
+          (reference "#PWR060") (unit 1)
         )
       )
@@
       (project "2.12 Mobile Robot"
         (path "/7775d959-b998-472b-ab8b-c8b5c0f34c21/3499523e-0988-447b-89ea-8d43c1ae7973"
-          (reference "#PWR045") (unit 1)
+          (reference "#PWR061") (unit 1)
         )
       )
@@
       (effects (font (size 1.27 1.27)) (justify left))
     )
-    (property "Footprint" "Resistor_SMD:R_0402_1005Metric" (at 131.826 89.789 90)
+    (property "Footprint" "Resistor_SMD:R_0201_0603Metric_Pad0.64x0.40mm_HandSolder" (at 131.826 89.789 90)
       (effects (font (size 1.27 1.27)) hide)
     )
@@
       (project "2.12 Mobile Robot"
         (path "/7775d959-b998-472b-ab8b-c8b5c0f34c21/3499523e-0988-447b-89ea-8d43c1ae7973"
-          (reference "R5") (unit 1)
-        )
-      )
+          (reference "R21") (unit 1)
+        )
+      )

Commit message: Made footprints from project libraries
Parts:
- Q1: footprint footprints:SOT95P285X140-6N -> 2.12_Mobile_Robot:SOT95P285X140-6N
- Q2: footprint footprints:SOT91P240X110-3N -> 2.12_Mobile_Robot:SOT91P240X110-3N
Changed lines of the file:
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@@
       (effects (font (size 1.27 1.27)))
     )
-    (property "Footprint" "footprints:SOT91P240X110-3N" (at 120.65 63.5 0)
+    (property "Footprint" "2.12_Mobile_Robot:SOT91P240X110-3N" (at 120.65 63.5 0)
       (effects (font (size 1.27 1.27)) (justify bottom) hide)
     )
@@
       (effects (font (size 1.27 1.27)) (justify left))
     )
-    (property "Footprint" "footprints:SOT95P285X140-6N" (at 115.57 73.66 0)
+    (property "Footprint" "2.12_Mobile_Robot:SOT95P285X140-6N" (at 115.57 73.66 0)
       (effects (font (size 1.27 1.27)) (justify bottom) hide)
     )
@@
       (effects (font (size 1.27 1.27)) (justify left))
     )
-    (property "Footprint" "footprints:SOT95P285X140-6N" (at 128.27 73.66 0)
-      (effects (font (size 1.27 1.27)) (justify bottom) hide)
-    )
+    (property "Footprint" "2.12_Mobile_Robot:SOT95P285X140-6N" (at 128.27 73.66 0)
+      (effects (font (size 1.27 1.27)) (justify bottom) hide)
+    )

Commit message: Added silkscreen callouts and fixed resistors
Parts:
- R7, R8: footprint Resistor_SMD:R_0201_0603Metric_Pad0.64x0.40mm_HandSolder -> Resistor_SMD:R_0603_1608Metric
Changed lines of the file:
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@@
       (effects (font (size 1.27 1.27)) (justify left))
     )
-    (property "Footprint" "Resistor_SMD:R_0201_0603Metric_Pad0.64x0.40mm_HandSolder" (at 114.046 89.154 90)
+    (property "Footprint" "Resistor_SMD:R_0603_1608Metric" (at 114.046 89.154 90)
       (effects (font (size 1.27 1.27)) hide)
     )
@@
       (effects (font (size 1.27 1.27)) (justify left))
     )
-    (property "Footprint" "Resistor_SMD:R_0201_0603Metric_Pad0.64x0.40mm_HandSolder" (at 131.826 89.789 90)
-      (effects (font (size 1.27 1.27)) hide)
-    )
+    (property "Footprint" "Resistor_SMD:R_0603_1608Metric" (at 131.826 89.789 90)
+      (effects (font (size 1.27 1.27)) hide)
+    )

Commit message: Tentatively ready for production
Parts:
- R7: footprint Resistor_SMD:R_0603_1608Metric -> footprint:0603_1608Metric; symbol Device:R_US -> jlcpcb-basic-resistor:0603,10k; LCSC (none) -> C25804; MFG (none) -> UNI-ROYAL(Uniroyal Elec); MFGPN (none) -> 0603WAF1002T5E
- R8: footprint Resistor_SMD:R_0603_1608Metric -> footprint:0603_1608Metric; symbol Device:R_US -> jlcpcb-basic-resistor:0603,47k; LCSC (none) -> C25819; MFG (none) -> UNI-ROYAL(Uniroyal Elec); MFGPN (none) -> 0603WAF4702T5E
Other:
- company: (none) -> MIT - jntaimo - Steve Banzaert
- title: (none) -> Zero Voltage Diode
Changed lines of the file:
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@@
 (kicad_sch (version 20230121) (generator eeschema)
   (paper "A4")
+  (title_block
+    (title "Zero Voltage Diode")
+    (company "MIT - jntaimo - Steve Banzaert")
+  )
   (junction (at 130.81 83.185) (diameter 0) (color 0 0 0 0)
   )
@@
     (stroke (width 0) (type default))
   )
+  (wire (pts (xy 113.03 91.44) (xy 113.03 92.71))
+    (stroke (width 0) (type default))
+  )
   (wire (pts (xy 123.19 83.185) (xy 130.81 83.185))
     (stroke (width 0) (type default))
@@
     (stroke (width 0) (type default))
   )
+  (wire (pts (xy 130.81 92.075) (xy 130.81 93.345))
+    (stroke (width 0) (type default))
+  )
   (wire (pts (xy 130.81 78.74) (xy 130.81 83.185))
     (stroke (width 0) (type default))
   )
-  (wire (pts (xy 113.03 83.82) (xy 113.03 85.09))
-    (stroke (width 0) (type default))
-  )
-  (wire (pts (xy 130.81 83.185) (xy 130.81 85.725))
+  (wire (pts (xy 113.03 83.82) (xy 113.03 86.36))
+    (stroke (width 0) (type default))
+  )
+  (wire (pts (xy 130.81 83.185) (xy 130.81 86.995))
     (stroke (width 0) (type default))
   )
@@
     )
   )
-  (symbol (lib_id "Device:R_US") (at 113.03 88.9 0) (unit 1)
+  (symbol (lib_id "jlcpcb-basic-resistor:0603,10k") (at 113.03 88.9 0) (unit 1)
     (in_bom yes) (on_board yes) (dnp no) (fields_autoplaced)
     (property "Reference" "R7" (at 115.57 88.265 0)
@@
       (effects (font (size 1.27 1.27)) (justify left))
     )
-    (property "Footprint" "Resistor_SMD:R_0603_1608Metric" (at 114.046 89.154 90)
-      (effects (font (size 1.27 1.27)) hide)
-    )
-    (property "Datasheet" "https://datasheet.lcsc.com/lcsc/2304140030_YAGEO-RC0402FR-0710KL_C60490.pdf" (at 113.03 88.9 0)
+    (property "Footprint" "footprint:0603_1608Metric" (at 113.03 88.9 0)
+      (effects (font (size 1.27 1.27)) hide)
+    )
+    (property "Datasheet" "https://datasheet.lcsc.com/lcsc/2110260030_UNI-ROYAL-Uniroyal-Elec-0603WAF1002T5E_C25804.pdf" (at 113.03 88.9 0)
       (effects (font (size 1.27 1.27)) hide)
     )
     (property "MPN" "C22548" (at 113.03 88.9 0)
       (effects (font (size 1.27 1.27)) hide)
+    )
+    (property "LCSC" "C25804" (at 113.03 88.9 0)
+      (effects (font (size 0 0)) hide)
+    )
+    (property "MFG" "UNI-ROYAL(Uniroyal Elec)" (at 113.03 88.9 0)
+      (effects (font (size 0 0)) hide)
+    )
+    (property "MFGPN" "0603WAF1002T5E" (at 113.03 88.9 0)
+      (effects (font (size 0 0)) hide)
     )
     (pin "1")
@@
     )
   )
-  (symbol (lib_id "Device:R_US") (at 130.81 89.535 0) (unit 1)
+  (symbol (lib_id "jlcpcb-basic-resistor:0603,47k") (at 130.81 89.535 0) (unit 1)
     (in_bom yes) (on_board yes) (dnp no) (fields_autoplaced)
     (property "Reference" "R8" (at 133.35 88.9 0)
@@
       (effects (font (size 1.27 1.27)) (justify left))
     )
-    (property "Footprint" "Resistor_SMD:R_0603_1608Metric" (at 131.826 89.789 90)
-      (effects (font (size 1.27 1.27)) hide)
-    )
-    (property "Datasheet" "~" (at 130.81 89.535 0)
+    (property "Footprint" "footprint:0603_1608Metric" (at 130.81 89.535 0)
+      (effects (font (size 1.27 1.27)) hide)
+    )
+    (property "Datasheet" "https://datasheet.lcsc.com/lcsc/2110260030_UNI-ROYAL-Uniroyal-Elec-0603WAF4702T5E_C25819.pdf" (at 130.81 89.535 0)
       (effects (font (size 1.27 1.27)) hide)
     )
@@
       (effects (font (size 1.27 1.27)) hide)
     )
-    (pin "1")
+    (property "LCSC" "C25819" (at 130.81 89.535 0)
+      (effects (font (size 0 0)) hide)
+    )
+    (property "MFG" "UNI-ROYAL(Uniroyal Elec)" (at 130.81 89.535 0)
+      (effects (font (size 0 0)) hide)
+    )
+    (property "MFGPN" "0603WAF4702T5E" (at 130.81 89.535 0)
+      (effects (font (size 0 0)) hide)
+    )
+    (pin "1")
